File: KiCad/EnvMon2.kicad_pcb (KiCad board)
At the start: 2 copper layers, 34 x 37 mm, 32 parts, among them J1 USB-C, J2 DC, J3 TEMP, M1 OLED1.5-RGB, U1 LMR16006+FB, U2 SCD41, U3 FT231XQ, U4 DS18B20, U5 ESP32-PICO-MINI-02, U6 QR

Commit message: Starting new code
Parts:
- R12: footprint Resistor_SMD:R_0603_1608Metric_Pad0.98x0.95mm_HandSolder -> RevK:R_0603
- R7: value 732R -> 680R
- R9: value 324R -> 220R
Changed lines of the file:
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@@
       (effects (font (size 0.5 0.5) (thickness 0.08)))
     )
-    (fp_text value "732R" (at 0 0 90) (layer "F.Fab")
+    (fp_text value "680R" (at 0 0 90) (layer "F.Fab")
       (effects (font (size 0.4 0.4) (thickness 0.08)))
     )
@@
     )
   )
-  (footprint "Resistor_SMD:R_0603_1608Metric_Pad0.98x0.95mm_HandSolder" (layer "F.Cu")
+  (footprint "RevK:R_0603" (layer "F.Cu")
     (at 132.5 91)
-    (descr "Resistor SMD 0603 (1608 Metric), square (rectangular) end terminal, IPC_7351 nominal with elongated pad for handsoldering. (Body size source: IPC-SM-782 page 72, https://www.pcb-3d.com/wordpress/wp-content/uploads/ipc-sm-782a_amendment_1_and_2.pdf), generated with kicad-footprint-generator")
-    (tags "resistor handsolder")
+    (descr "Capacitor SMD 0603 (1608 Metric), square (rectangular) end terminal, IPC_7351 nominal, (Body size source: IPC-SM-782 page 76, https://www.pcb-3d.com/wordpress/wp-content/uploads/ipc-sm-782a_amendment_1_and_2.pdf), generated with kicad-footprint-generator")
+    (tags "capacitor")
     (property "Sheetfile" "EnvMon2.kicad_sch")
     (property "Sheetname" "")
     (attr smd)
-    (fp_text reference "R12" (at 0 -1.43) (layer "F.SilkS") hide
-      (effects (font (size 1 1) (thickness 0.15)))
-    )
-    (fp_text value "4k7" (at 0 1.43) (layer "F.Fab")
-      (effects (font (size 1 1) (thickness 0.15)))
-    )
-    (fp_text user "${REFERENCE}" (at 0 0) (layer "F.Fab")
+    (fp_text reference "R12" (at -1.6 0 90) (layer "F.SilkS") hide
+      (effects (font (size 0.5 0.5) (thickness 0.08)))
+    )
+    (fp_text value "4k7" (at 0 0) (layer "F.Fab")
+      (effects (font (size 0.4 0.4) (thickness 0.08)))
+    )
+    (fp_text user "${REFERENCE}" (at 0 -0.8) (layer "F.Fab")
       (effects (font (size 0.4 0.4) (thickness 0.06)))
     )
-    (fp_line (start -0.254724 0.5225) (end 0.254724 0.5225) (layer "F.SilkS") (width 0.12))
-    (fp_line (start -0.254724 -0.5225) (end 0.254724 -0.5225) (layer "F.SilkS") (width 0.12))
-    (fp_line (start 1.65 0.73) (end -1.65 0.73) (layer "F.CrtYd") (width 0.05))
-    (fp_line (start -1.65 -0.73) (end 1.65 -0.73) (layer "F.CrtYd") (width 0.05))
-    (fp_line (start -1.65 0.73) (end -1.65 -0.73) (layer "F.CrtYd") (width 0.05))
-    (fp_line (start 1.65 -0.73) (end 1.65 0.73) (layer "F.CrtYd") (width 0.05))
-    (fp_line (start 0.8 0.4125) (end -0.8 0.4125) (layer "F.Fab") (width 0.1))
-    (fp_line (start 0.8 -0.4125) (end 0.8 0.4125) (layer "F.Fab") (width 0.1))
-    (fp_line (start -0.8 0.4125) (end -0.8 -0.4125) (layer "F.Fab") (width 0.1))
-    (fp_line (start -0.8 -0.4125) (end 0.8 -0.4125) (layer "F.Fab") (width 0.1))
-    (pad "1" smd roundrect (at -0.9125 0) (size 0.975 0.95) (layers "F.Cu" "F.Paste" "F.Mask") (roundrect_rratio 0.25)
+    (fp_line (start -0.3 -0.5) (end 0.3 -0.5) (layer "F.SilkS") (width 0.12))
+    (fp_line (start -0.3 0.5) (end 0.3 0.5) (layer "F.SilkS") (width 0.12))
+    (fp_line (start 0.8 0.4) (end -0.8 0.4) (layer "F.CrtYd") (width 0.05))
+    (fp_line (start -0.8 0.4) (end -0.8 -0.4) (layer "F.CrtYd") (width 0.05))
+    (fp_line (start -0.8 -0.4) (end 0.8 -0.4) (layer "F.CrtYd") (width 0.05))
+    (fp_line (start 0.8 -0.4) (end 0.8 0.4) (layer "F.CrtYd") (width 0.05))
+    (fp_line (start -0.8 0.4) (end -0.8 -0.4) (layer "F.Fab") (width 0.1))
+    (fp_line (start 0.8 0.4) (end -0.8 0.4) (layer "F.Fab") (width 0.1))
+    (fp_line (start -0.8 -0.4) (end 0.8 -0.4) (layer "F.Fab") (width 0.1))
+    (fp_line (start 0.8 -0.4) (end 0.8 0.4) (layer "F.Fab") (width 0.1))
+    (pad "1" smd roundrect (at -0.825 0) (size 0.8 0.95) (layers "F.Cu" "F.Paste" "F.Mask") (roundrect_rratio 0.25)
       (net 12 "+3V3") (pintype "passive"))
-    (pad "2" smd roundrect (at 0.9125 0) (size 0.975 0.95) (layers "F.Cu" "F.Paste" "F.Mask") (roundrect_rratio 0.25)
+    (pad "2" smd roundrect (at 0.825 0) (size 0.8 0.95) (layers "F.Cu" "F.Paste" "F.Mask") (roundrect_rratio 0.25)
       (net 9 "TEMP") (pintype "passive"))
-    (model "${KICAD6_3DMODEL_DIR}/Resistor_SMD.3dshapes/R_0603_1608Metric.wrl"
+    (model "${KICAD6_3DMODEL_DIR}/Resistor_SMD.3dshapes/R_0603_1608Metric.step"
       (offset (xyz 0 0 0))
       (scale (xyz 1 1 1))
@@
       (effects (font (size 0.5 0.5) (thickness 0.08)))
     )
-    (fp_text value "324R" (at 0 0) (layer "F.Fab")
+    (fp_text value "220R" (at 0 0) (layer "F.Fab")
       (effects (font (size 0.4 0.4) (thickness 0.08)))
     )
@@
     (property "Sheetfile" "EnvMon2.kicad_sch")
     (property "Sheetname" "")
+    (property "exclude_from_bom" "")
     (attr exclude_from_pos_files exclude_from_bom)
     (fp_text reference "Logo1" (at 0 -5) (layer "B.SilkS") hide

Commit message: New case
Parts:
- removed U6: QR, RevK:QR-ENVMON
- added Logo2: AJK, RevK:AJK, F.Cu at (113.5, 72.0)
- R12: value 4k7 -> 10k
- R13: value 10k -> 4k7
- R3, R4: footprint Resistor_SMD:R_0603_1608Metric_Pad0.98x0.95mm_HandSolder -> RevK:R_0603
- U4: value DS18B20 -> ESP32-PICO-MINI-02; footprint Package_TO_SOT_THT:TO-92_Inline -> RevK:ESP32-PICO-MINI-02
- U5: value ESP32-PICO-MINI-02 -> QR; footprint RevK:ESP32-PICO-MINI-02 -> RevK:QR-ENVMON; moved to B.Cu
- moved U4 42.6 mm to (128.0, 68.7), turned to 0 degrees
- moved M1 29.3 mm to (144.5, 63.0)
- moved U2 28.7 mm to (105.5, 57.5), turned to 90 degrees
- moved C3 28.6 mm to (135.8, 77.3), turned to 0 degrees
- moved R12 26.2 mm to (119.6, 68.2), turned to -90 degrees
- moved L1 25.2 mm to (132.2, 78.8), turned to 90 degrees
- moved D1 24.3 mm to (135.4, 80.4), turned to 90 degrees
- moved D3 21.4 mm to (137.0, 64.6), turned to 180 degrees
- moved C2 20.6 mm to (135.8, 83.5), turned to 0 degrees
- moved R13 20.4 mm to (111.4, 91.0), turned to 0 degrees
- moved R9 20.0 mm to (137.0, 67.4), turned to 180 degrees
- moved U5 19.8 mm to (122.2, 97.0), turned to 0 degrees
- moved U1 19.8 mm to (132.2, 82.7), turned to 90 degrees
- moved R4 19.7 mm to (124.6, 91.8)
- moved J1 19.6 mm to (122.2, 100.0)
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Connections:
- R12 pad 2: TEMP -> EN
- R13 pad 1: +3V3 -> TEMP
- R13 pad 2: EN -> +3V3
- U2 pad 19: unconnected-(U2-Pad19) -> +3V3
- U4 pad 2: TEMP -> GND
Routing:
- net CO2-SDA: track 14.6 -> 37.1 mm
- net CO2-SCL: track 20.1 -> 38.6 mm
- net O: track 13.0 -> 30.5 mm
- net I: track 7.43 -> 24.5 mm, vias 0 -> 2
- net OLED-MOSI: track 7.25 -> 24.2 mm
- net TEMP: track 45.9 -> 29.5 mm, vias 2 -> 0
- net OLED-SCLK: track 10.2 -> 25.7 mm
- net OLED-CS0: track 12.8 -> 27.9 mm
- net OLED-RST: track 18.6 -> 31.9 mm, vias 1 -> 0
- net OLED-DC: track 16.5 -> 29.9 mm, vias 1 -> 0
- net GND: track 28.6 -> 36.2 mm
- net DC: track 26.0 -> 19.1 mm, vias 2 -> 0
- net +3V3: track 131.5 -> 136.5 mm, vias 5 -> 3
- net Net-(R10-Pad2): track 13.4 -> 8.51 mm, vias 2 -> 0
- net BOOT: track 13.6 -> 18.0 mm
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Other:
- board size 34 x 37 mm -> 44.5 x 48 mm
- board text added: "DC 4V-60V"
- board text added: "DS18B20"
- board text removed: "DC"
- board text removed: "GND"

Commit message: Redesign
Parts:
- moved U2 17.4 mm to (92.0, 68.5), turned to 180 degrees
- moved Logo2 15.4 mm to (116.2, 87.1)
- moved U4 7.79 mm to (122.2, 73.9)
- moved R12 6.18 mm to (115.0, 72.3)
- moved U3 0.45 mm to (122.0, 85.2)
- moved C4 0.40 mm to (128.2, 88.7)
- moved R10 0.40 mm to (127.0, 88.7)
- moved R11 0.40 mm to (125.8, 88.7)
Routing:
- net CO2-SCL: track 38.6 -> 52.5 mm
- net GND: track 36.2 -> 50.0 mm, vias 3 -> 7
- net CO2-SDA: track 37.1 -> 48.6 mm, vias 2 -> 4
- net BOOT: track 18.0 -> 7.79 mm, vias 2 -> 0
- net I: track 24.5 -> 14.8 mm
- net R: track 3.70 -> 13.4 mm
- net B: track 4.03 -> 13.4 mm
- net OLED-RST: track 31.9 -> 22.6 mm
- net G: track 2.32 -> 11.4 mm
- net OLED-DC: track 29.9 -> 21.1 mm
- net OLED-SCLK: track 25.7 -> 17.2 mm
- net OLED-CS0: track 27.9 -> 19.6 mm
- net OLED-MOSI: track 24.2 -> 15.9 mm
- net +3V3: track 136.5 -> 128.5 mm
- net TEMP: track 29.5 -> 21.8 mm
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Other:
- board size 44.5 x 48 mm -> 58 x 37 mm

Commit message: Tidy
Parts:
- moved Logo1 24.2 mm to (134.8, 83.9)
Other:
- outline, holes or cut-outs redrawn
Changed lines of the file:
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@@
   )
   (footprint "RevK:AJK" (layer "B.Cu")
-    (at 110.9 79.5 180)
+    (at 134.75 83.875 180)
     (property "Note" "Non part, PCB printed")
     (property "Sheetfile" "EnvMon2.kicad_sch")
@@
     )
   )
-  (gr_line (start 100 74) (end 86.5 74) (layer "Edge.Cuts") (width 0.05))
+  (gr_line (start 99 74) (end 87.5 74) (layer "Edge.Cuts") (width 0.05))
   (gr_arc (start 97.5 64.5) (mid 98.5 63.5) (end 99.5 64.5) (layer "Edge.Cuts") (width 0.05))
   (gr_line (start 134.5 67.25) (end 134.5 63) (layer "Edge.Cuts") (width 0.05))
   (gr_arc (start 112 73.5) (mid 113.237437 74.012563) (end 113.75 75.25) (layer "Edge.Cuts") (width 0.05))
   (gr_line (start 106 68.25) (end 133.5 68.25) (layer "Edge.Cuts") (width 0.05))
+  (gr_arc (start 86.5 64) (mid 86.792893 63.292893) (end 87.5 63) (layer "Edge.Cuts") (width 0.05))
   (gr_arc (start 106 68.25) (mid 105.292893 67.957107) (end 105 67.25) (layer "Edge.Cuts") (width 0.05))
   (gr_arc (start 134.5 67.25) (mid 134.207107 67.957107) (end 133.5 68.25) (layer "Edge.Cuts") (width 0.05))
-  (gr_line (start 86.5 74) (end 86.5 63) (layer "Edge.Cuts") (width 0.05))
+  (gr_line (start 86.5 73) (end 86.5 64) (layer "Edge.Cuts") (width 0.05))
   (gr_line (start 100 100) (end 144.5 100) (layer "Edge.Cuts") (width 0.05))
   (gr_line (start 97.5 64.5) (end 97.5 72.5) (layer "Edge.Cuts") (width 0.05))
+  (gr_arc (start 87.5 74) (mid 86.792893 73.707107) (end 86.5 73) (layer "Edge.Cuts") (width 0.05))
   (gr_line (start 144.5 100) (end 144.5 63) (layer "Edge.Cuts") (width 0.05))
   (gr_arc (start 106.25 78.5) (mid 105.012563 77.987437) (end 104.5 76.75) (layer "Edge.Cuts") (width 0.05))
@@
   (gr_arc (start 102.5 72.5) (mid 100.75 70.75) (end 102.5 69) (layer "Edge.Cuts") (width 0.05))
   (gr_arc (start 112 69) (mid 113.75 70.75) (end 112 72.5) (layer "Edge.Cuts") (width 0.05))
-  (gr_line (start 105 63) (end 86.5 63) (layer "Edge.Cuts") (width 0.05))
+  (gr_line (start 105 63) (end 87.5 63) (layer "Edge.Cuts") (width 0.05))
   (gr_line (start 104.5 75.25) (end 104.5 76.75) (layer "Edge.Cuts") (width 0.05))
   (gr_arc (start 99.5 72.5) (mid 98.5 73.5) (end 97.5 72.5) (layer "Edge.Cuts") (width 0.05))
-  (gr_line (start 100 74) (end 100 100) (layer "Edge.Cuts") (width 0.05))
+  (gr_line (start 100 75) (end 100 100) (layer "Edge.Cuts") (width 0.05))
   (gr_arc (start 113.75 76.75) (mid 113.237437 77.987437) (end 112 78.5) (layer "Edge.Cuts") (width 0.05))
+  (gr_arc (start 99 74) (mid 99.707107 74.292893) (end 100 75) (layer "Edge.Cuts") (width 0.05))
   (gr_line (start 105 63) (end 105 67.25) (layer "Edge.Cuts") (width 0.05))
   (gr_text "DC\n4V-60V" (at 135.5 97) (layer "B.SilkS")
     (effects (font (size 1 1) (thickness 0.15)) (justify mirror))
   )
-  (gr_text "Environmental\nMonitor" (at 111.5 74.625) (layer "B.SilkS")
+  (gr_text "Environmental\nMonitor" (at 135.25 78.5) (layer "B.SilkS")
     (effects (font (size 1 1) (thickness 0.15)) (justify mirror))
   )

Commit message: Silkscreen
Routing:
- net GND: vias 7 -> 6
Other:
- board text added: "14"
- board text added: "25"
- board text added: "26"
- board text added: "27"
- board text added: "3.3"
- board text added: "32"
- board text added: "33"
- board text added: "CO₂"
- board text added: "LED: 7/19/8"
- board text added: "SCD41 SCL: 21 SDA: 22"
- board text added: "⏚"
Changed lines of the file:
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@@
     (effects (font (size 1 1) (thickness 0.15)) (justify mirror))
+  )
+  (gr_text "33" (at 100.838 81.534 90) (layer "B.SilkS")
+    (effects (font (size 0.75 0.75) (thickness 0.15)) (justify mirror))
+  )
+  (gr_text "⏚" (at 100.838 76.454 90) (layer "B.SilkS")
+    (effects (font (size 0.75 0.75) (thickness 0.15)) (justify mirror))
+  )
+  (gr_text "SCD41\nSCL: 21\nSDA: 22" (at 92 71) (layer "B.SilkS")
+    (effects (font (size 0.75 0.75) (thickness 0.15)) (justify mirror))
   )
   (gr_text "Environmental\nMonitor" (at 135.25 78.5) (layer "B.SilkS")
     (effects (font (size 1 1) (thickness 0.15)) (justify mirror))
   )
+  (gr_text "3.3" (at 100.838 73.914 90) (layer "B.SilkS")
+    (effects (font (size 0.75 0.75) (thickness 0.15)) (justify mirror))
+  )
+  (gr_text "CO₂" (at 92 66.25) (layer "B.SilkS")
+    (effects (font (size 2 2) (thickness 0.3)) (justify mirror))
+  )
+  (gr_text "25" (at 100.838 84.074 90) (layer "B.SilkS")
+    (effects (font (size 0.75 0.75) (thickness 0.15)) (justify mirror))
+  )
   (gr_text "DS18B20" (at 110.25 97.75) (layer "B.SilkS")
     (effects (font (size 1 1) (thickness 0.15)) (justify mirror))
+  )
+  (gr_text "14" (at 110.25 91.75) (layer "B.SilkS")
+    (effects (font (size 0.75 0.75) (thickness 0.15)) (justify mirror))
+  )
+  (gr_text "32" (at 100.838 78.994 90) (layer "B.SilkS")
+    (effects (font (size 0.75 0.75) (thickness 0.15)) (justify mirror))
+  )
+  (gr_text "26" (at 100.838 86.614 90) (layer "B.SilkS")
+    (effects (font (size 0.75 0.75) (thickness 0.15)) (justify mirror))
+  )
+  (gr_text "27" (at 100.838 89.154 90) (layer "B.SilkS")
+    (effects (font (size 0.75 0.75) (thickness 0.15)) (justify mirror))
+  )
+  (gr_text "LED: 7/19/8" (at 140.5 68.75) (layer "B.SilkS")
+    (effects (font (size 0.75 0.75) (thickness 0.15)) (justify mirror))
   )
   (gr_text "Environmental\nMonitor" (at 141 80.75 90) (layer "F.SilkS")
@@
   (segment (start 94.5 71) (end 93.2 69.7) (width 0.5) (layer "F.Cu") (net 11))
   (segment (start 121.05 87.15) (end 121.05 87.2) (width 0.25) (layer "F.Cu") (net 11))
-  (via (at 100.5 72.75) (size 0.8) (drill 0.4) (layers "F.Cu" "B.Cu") (free) (net 11))
   (via (at 88 72.4) (size 0.8) (drill 0.4) (layers "F.Cu" "B.Cu") (free) (net 11))
   (via (at 92 68.5) (size 0.8) (drill 0.4) (layers "F.Cu" "B.Cu") (net 11))
