File: KiCad/EnvMon2.kicad_sch (KiCad schematic)
At the start: 30 parts, among them J1 USB-C, J2 DC, J3 TEMP, M1 OLED1.5-RGB, U1 LMR16006+FB, U2 SCD41, U3 FT231XQ, U4 DS18B20, U5 ESP32-PICO-MINI-02, U6 QR

Commit message: Tidy
Parts:
- added R5, R6: 27R, RevK:R_0603, symbol Device:R
- J1: symbol Connector:USB_C_Receptacle_USB2.0 -> RevK:USB-C
- U3: footprint Package_DFN_QFN:QFN-20-1EP_4x4mm_P0.5mm_EP2.5x2.5mm -> RevK:QFN-20-1EP_4x4mm_P0.5mm_EP2.5x2.5mm; symbol Interface_USB:FT231XQ -> RevK:FT231XQ
- renumbered R8 to R10, R9 to R11, R10 to R12, R11 to R13, R5 to R7, R6 to R8, R7 to R9
Connections:
- net CO2-SCL: now also U5.15 (IO25)
- net CO2-SDA: now also U5.16 (IO26)
- net D+: now also R6.2; no longer J1.A6 (D+), J1.B6 (D+)
- net D-: now also R5.2; no longer J1.A7 (D-), J1.B7 (D-)
- new net: J1.A6 (D+), J1.B6 (D+), R6.1
- new net: J1.A7 (D-), J1.B7 (D-), R5.1
- now unconnected: U2.1 (DNC), U2.11 (DNC), U2.12 (DNC), U2.13 (DNC), U2.14 (DNC), U2.15 (DNC), U2.16 (DNC), U2.17 (DNC), U2.18 (DNC), U2.2 (DNC), U2.3 (DNC), U2.4 (DNC), U2.5 (DNC), U2.8 (DNC)
- no-connect marks 6 -> 17
Changed lines of the file:
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@@
   (no_connect (at 149.86 50.8))
   (no_connect (at 149.86 53.34))
-  (no_connect (at 55.88 55.88))
+  (no_connect (at 226.06 73.66))
+  (no_connect (at 226.06 78.74))
+  (no_connect (at 226.06 76.2))
+  (no_connect (at 195.58 48.26))
+  (no_connect (at 195.58 45.72))
+  (no_connect (at 195.58 43.18))
+  (no_connect (at 195.58 53.34))
+  (no_connect (at 195.58 50.8))
+  (no_connect (at 195.58 40.64))
+  (no_connect (at 195.58 60.96))
+  (no_connect (at 195.58 66.04))
+  (no_connect (at 195.58 73.66))
+  (no_connect (at 226.06 58.42))
   (no_connect (at 58.42 99.06))
-  (no_connect (at 55.88 58.42))
   (wire (pts (xy 55.88 33.02) (xy 58.42 33.02))
     (stroke (width 0) (type default) (color 0 0 0 0))
@@
     )
   )
-  (global_label "CO2-SCL" (shape input) (at 182.88 104.14 180) (fields_autoplaced)
-    (effects (font (size 1.27 1.27)) (justify right))
-    (property "Intersheet References" "${INTERSHEET_REFS}" (id 0) (at 133.985 -17.145 0)
+  (global_label "CO2-SCL" (shape input) (at 226.06 68.58 0) (fields_autoplaced)
+    (effects (font (size 1.27 1.27)) (justify left))
+    (property "Intersheet References" "${INTERSHEET_REFS}" (id 0) (at 274.955 189.865 0)
       (effects (font (size 1.27 1.27)) hide)
     )
@@
     )
   )
-  (global_label "D-" (shape bidirectional) (at 58.42 40.64 0) (fields_autoplaced)
+  (global_label "D-" (shape bidirectional) (at 66.04 40.64 0) (fields_autoplaced)
     (effects (font (size 1.27 1.27)) (justify left))
-    (property "Intersheet References" "${INTERSHEET_REFS}" (id 0) (at 63.5866 40.5606 0)
+    (property "Intersheet References" "${INTERSHEET_REFS}" (id 0) (at 71.2066 40.5606 0)
       (effects (font (size 1.27 1.27)) (justify left) hide)
     )
@@
     )
   )
-  (global_label "CO2-SDA" (shape input) (at 182.88 101.6 180) (fields_autoplaced)
-    (effects (font (size 1.27 1.27)) (justify right))
-    (property "Intersheet References" "${INTERSHEET_REFS}" (id 0) (at 133.985 -22.225 0)
+  (global_label "CO2-SDA" (shape input) (at 226.06 71.12 0) (fields_autoplaced)
+    (effects (font (size 1.27 1.27)) (justify left))
+    (property "Intersheet References" "${INTERSHEET_REFS}" (id 0) (at 274.955 194.945 0)
       (effects (font (size 1.27 1.27)) hide)
     )
@@
     )
   )
-  (global_label "D+" (shape bidirectional) (at 58.42 48.26 0) (fields_autoplaced)
+  (global_label "D+" (shape bidirectional) (at 66.04 48.26 0) (fields_autoplaced)
     (effects (font (size 1.27 1.27)) (justify left))
-    (property "Intersheet References" "${INTERSHEET_REFS}" (id 0) (at 63.5866 48.1806 0)
+    (property "Intersheet References" "${INTERSHEET_REFS}" (id 0) (at 71.2066 48.1806 0)
       (effects (font (size 1.27 1.27)) (justify left) hide)
     )
@@
     )
   )
-  (symbol (lib_id "Connector:USB_C_Receptacle_USB2.0") (at 40.64 43.18 0) (unit 1)
+  (symbol (lib_id "RevK:USB-C") (at 40.64 43.18 0) (unit 1)
     (in_bom yes) (on_board yes)
     (property "Reference" "J1" (id 0) (at 43.3578 21.1582 0))
@@
     )
   )
-  (symbol (lib_id "Interface_USB:FT231XQ") (at 132.08 43.18 0) (unit 1)
+  (symbol (lib_id "RevK:FT231XQ") (at 132.08 43.18 0) (unit 1)
     (in_bom yes) (on_board yes)
     (property "Reference" "U3" (id 0) (at 119.38 66.04 0))
     (property "Value" "FT231XQ" (id 1) (at 129.54 52.07 0))
-    (property "Footprint" "Package_DFN_QFN:QFN-20-1EP_4x4mm_P0.5mm_EP2.5x2.5mm" (id 2) (at 166.37 63.5 0)
+    (property "Footprint" "RevK:QFN-20-1EP_4x4mm_P0.5mm_EP2.5x2.5mm" (id 2) (at 166.37 63.5 0)
       (effects (font (size 1.27 1.27)) hide)
     )
@@
   (symbol (lib_id "Device:R") (at 113.03 142.24 270) (unit 1)
     (in_bom yes) (on_board yes)
-    (property "Reference" "R7" (id 0) (at 113.03 144.145 90))
+    (property "Reference" "R9" (id 0) (at 113.03 144.145 90))
     (property "Value" "324R" (id 1) (at 113.03 142.24 90))
     (property "Footprint" "RevK:R_0603" (id 2) (at 113.03 140.462 90)
@@
   (symbol (lib_id "Device:R") (at 113.03 132.08 270) (unit 1)
     (in_bom yes) (on_board yes)
-    (property "Reference" "R5" (id 0) (at 113.03 133.985 90))
+    (property "Reference" "R7" (id 0) (at 113.03 133.985 90))
     (property "Value" "732R" (id 1) (at 113.03 132.08 90))
     (property "Footprint" "RevK:R_0603" (id 2) (at 113.03 130.302 90)
@@
   (symbol (lib_id "Device:R") (at 113.03 137.16 270) (unit 1)
     (in_bom yes) (on_board yes)
-    (property "Reference" "R6" (id 0) (at 113.03 139.065 90))
+    (property "Reference" "R8" (id 0) (at 113.03 139.065 90))
     (property "Value" "2K" (id 1) (at 113.03 137.16 90))
     (property "Footprint" "RevK:R_0603" (id 2) (at 113.03 135.382 90)
@@
       (effects (font (size 1.27 1.27)) (justify right))
     )
-    (property "Value" "DC" (id 1) (at 57.785 121.285 0)
+    (property "Value" "DC" (id 1) (at 63.5 121.92 0)
       (effects (font (size 1.27 1.27)) (justify right))
     )
@@
   (symbol (lib_id "Device:R") (at 168.91 127 90) (unit 1)
     (in_bom yes) (on_board yes)
-    (property "Reference" "R10" (id 0) (at 170.18 124.46 90)
+    (property "Reference" "R12" (id 0) (at 170.18 124.46 90)
       (effects (font (size 1.27 1.27)) (justify left))
     )
@@
     (pin "2")
   )
+  (symbol (lib_id "Device:R") (at 62.23 48.26 90) (unit 1)
+    (in_bom yes) (on_board yes)
+    (property "Reference" "R6" (id 0) (at 60.96 50.8 90))
+    (property "Value" "27R" (id 1) (at 62.23 48.26 90))
+    (property "Footprint" "RevK:R_0603" (id 2) (at 62.23 50.038 90)
+      (effects (font (size 1.27 1.27)) hide)
+    )
+    (property "Datasheet" "~" (id 3) (at 62.23 48.26 0)
+      (effects (font (size 1.27 1.27)) hide)
+    )
+    (pin "1")
+    (pin "2")
+  )
   (symbol (lib_id "RevK:LMR16006+FB") (at 49.53 131.445 0) (unit 1)
     (in_bom yes) (on_board yes)
@@
   (symbol (lib_id "Device:R") (at 193.04 34.29 0) (unit 1)
     (in_bom yes) (on_board yes)
-    (property "Reference" "R11" (id 0) (at 194.945 34.29 90))
+    (property "Reference" "R13" (id 0) (at 194.945 34.29 90))
     (property "Value" "10k" (id 1) (at 193.04 34.29 90))
     (property "Footprint" "RevK:R_0603" (id 2) (at 191.262 34.29 90)
@@
   (symbol (lib_id "Device:R") (at 160.02 62.23 0) (unit 1)
     (in_bom yes) (on_board yes)
-    (property "Reference" "R9" (id 0) (at 161.925 62.23 90))
+    (property "Reference" "R11" (id 0) (at 161.925 62.23 90))
     (property "Value" "10k" (id 1) (at 160.02 62.23 90))
     (property "Footprint" "RevK:R_0603" (id 2) (at 158.242 62.23 90)
@@
     (pin "1")
   )
+  (symbol (lib_id "Device:R") (at 62.23 40.64 90) (unit 1)
+    (in_bom yes) (on_board yes)
+    (property "Reference" "R5" (id 0) (at 60.96 43.18 90))
+    (property "Value" "27R" (id 1) (at 62.23 40.64 90))
+    (property "Footprint" "RevK:R_0603" (id 2) (at 62.23 42.418 90)
+      (effects (font (size 1.27 1.27)) hide)
+    )
+    (property "Datasheet" "~" (id 3) (at 62.23 40.64 0)
+      (effects (font (size 1.27 1.27)) hide)
+    )
+    (pin "1")
+    (pin "2")
+  )
   (symbol (lib_id "Device:R") (at 49.53 145.415 180) (unit 1)
     (in_bom yes) (on_board yes)
@@
   (symbol (lib_id "Device:R") (at 160.02 54.61 0) (unit 1)
     (in_bom yes) (on_board yes)
-    (property "Reference" "R8" (id 0) (at 161.925 54.61 90))
+    (property "Reference" "R10" (id 0) (at 161.925 54.61 90))
     (property "Value" "4k7" (id 1) (at 160.02 54.61 90))
     (property "Footprint" "RevK:R_0603" (id 2) (at 158.242 54.61 90)
@@
       (reference "R4") (unit 1) (value "5K1") (footprint "Resistor_SMD:R_0603_1608Metric_Pad0.98x0.95mm_HandSolder")
     )
+    (path "/d9ede1d9-98fb-4bf6-9188-b8434de8eed0"
+      (reference "R5") (unit 1) (value "27R") (footprint "RevK:R_0603")
+    )
+    (path "/64e3fa84-8672-4bfb-a08c-14181f58ca5f"
+      (reference "R6") (unit 1) (value "27R") (footprint "RevK:R_0603")
+    )
     (path "/00000000-0000-0000-0000-000060cf9e4d"
-      (reference "R5") (unit 1) (value "732R") (footprint "RevK:R_0603")
+      (reference "R7") (unit 1) (value "732R") (footprint "RevK:R_0603")
     )
     (path "/00000000-0000-0000-0000-000060cfbfaf"
-      (reference "R6") (unit 1) (value "2K") (footprint "RevK:R_0603")
+      (reference "R8") (unit 1) (value "2K") (footprint "RevK:R_0603")
     )
     (path "/00000000-0000-0000-0000-000060a436c8"
-      (reference "R7") (unit 1) (value "324R") (footprint "RevK:R_0603")
+      (reference "R9") (unit 1) (value "324R") (footprint "RevK:R_0603")
     )
     (path "/e7149988-8da9-4254-8dc1-168b761f2899"
-      (reference "R8") (unit 1) (value "4k7") (footprint "RevK:R_0603")
+      (reference "R10") (unit 1) (value "4k7") (footprint "RevK:R_0603")
     )
     (path "/ae993647-4c98-4bb9-8c7a-3beaf65656f4"
-      (reference "R9") (unit 1) (value "10k") (footprint "RevK:R_0603")
+      (reference "R11") (unit 1) (value "10k") (footprint "RevK:R_0603")
     )
     (path "/40905c56-15f1-4710-87cf-81fb9e340012"
-      (reference "R10") (unit 1) (value "4k7") (footprint "Resistor_SMD:R_0603_1608Metric_Pad0.98x0.95mm_HandSolder")
+      (reference "R12") (unit 1) (value "4k7") (footprint "Resistor_SMD:R_0603_1608Metric_Pad0.98x0.95mm_HandSolder")
     )
     (path "/90b8eaac-a159-4dee-976f-dbdad4d50f22"
-      (reference "R11") (unit 1) (value "10k") (footprint "RevK:R_0603")
+      (reference "R13") (unit 1) (value "10k") (footprint "RevK:R_0603")
     )
     (path "/7cbfa237-177e-4c8c-8cb5-2871c201d869"
@@
     )
     (path "/00000000-0000-0000-0000-00006081e5c7"
-      (reference "U3") (unit 1) (value "FT231XQ") (footprint "Package_DFN_QFN:QFN-20-1EP_4x4mm_P0.5mm_EP2.5x2.5mm")
+      (reference "U3") (unit 1) (value "FT231XQ") (footprint "RevK:QFN-20-1EP_4x4mm_P0.5mm_EP2.5x2.5mm")
     )
     (path "/317f5b5b-00a7-424d-ad37-e0c1b6da4c8d"

Commit message: Starting new code
Parts:
- Logo1: now left out of the parts list
- R12: footprint Resistor_SMD:R_0603_1608Metric_Pad0.98x0.95mm_HandSolder -> RevK:R_0603
- R7: value 732R -> 680R
- R9: value 324R -> 220R
Changed lines of the file:
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@@
   )
   (symbol (lib_id "RevK:AJK") (at 272.415 175.895 0) (unit 1)
-    (in_bom yes) (on_board yes)
+    (in_bom no) (on_board yes)
     (property "Reference" "Logo1" (id 0) (at 273.05 174.7266 0)
       (effects (font (size 1.27 1.27)) (justify left) hide)
@@
     (in_bom yes) (on_board yes)
     (property "Reference" "R9" (id 0) (at 113.03 144.145 90))
-    (property "Value" "324R" (id 1) (at 113.03 142.24 90))
+    (property "Value" "220R" (id 1) (at 113.03 142.24 90))
     (property "Footprint" "RevK:R_0603" (id 2) (at 113.03 140.462 90)
       (effects (font (size 1.27 1.27)) hide)
@@
     (in_bom yes) (on_board yes)
     (property "Reference" "R7" (id 0) (at 113.03 133.985 90))
-    (property "Value" "732R" (id 1) (at 113.03 132.08 90))
+    (property "Value" "680R" (id 1) (at 113.03 132.08 90))
     (property "Footprint" "RevK:R_0603" (id 2) (at 113.03 130.302 90)
       (effects (font (size 1.27 1.27)) hide)
@@
       (effects (font (size 1.27 1.27)) (justify left))
     )
-    (property "Footprint" "Resistor_SMD:R_0603_1608Metric_Pad0.98x0.95mm_HandSolder" (id 2) (at 168.91 128.778 90)
+    (property "Footprint" "RevK:R_0603" (id 2) (at 168.91 128.778 90)
       (effects (font (size 1.27 1.27)) hide)
     )
@@
     )
     (path "/00000000-0000-0000-0000-000060cf9e4d"
-      (reference "R7") (unit 1) (value "732R") (footprint "RevK:R_0603")
+      (reference "R7") (unit 1) (value "680R") (footprint "RevK:R_0603")
     )
     (path "/00000000-0000-0000-0000-000060cfbfaf"
@@
     )
     (path "/00000000-0000-0000-0000-000060a436c8"
-      (reference "R9") (unit 1) (value "324R") (footprint "RevK:R_0603")
+      (reference "R9") (unit 1) (value "220R") (footprint "RevK:R_0603")
     )
     (path "/e7149988-8da9-4254-8dc1-168b761f2899"
@@
     )
     (path "/40905c56-15f1-4710-87cf-81fb9e340012"
-      (reference "R12") (unit 1) (value "4k7") (footprint "Resistor_SMD:R_0603_1608Metric_Pad0.98x0.95mm_HandSolder")
+      (reference "R12") (unit 1) (value "4k7") (footprint "RevK:R_0603")
     )
     (path "/90b8eaac-a159-4dee-976f-dbdad4d50f22"

Commit message: New case
Parts:
- removed U4: DS18B20, Package_TO_SOT_THT:TO-92_Inline, symbol Sensor_Temperature:DS18B20
- added Logo1: AJK, RevK:AJK, symbol RevK:AJK
- R3, R4: footprint Resistor_SMD:R_0603_1608Metric_Pad0.98x0.95mm_HandSolder -> RevK:R_0603
- renumbered Logo1 to Logo2, R13 to R12, R12 to R13, U5 to U4, U6 to U5
Connections:
- net +3V3: now also R13.2, U2.19 (VDDH); no longer R13.1
- net B: now also U4.28 (IO8); no longer U4.21 (IO15)
- net CO2-SCL: now also U4.35 (IO21); no longer U4.15 (IO25)
- net CO2-SDA: now also U4.34 (IO22); no longer U4.16 (IO26)
- net G: now also U4.33 (IO19); no longer U4.18 (IO14)
- net OLED-CS0: now also U4.15 (IO25); no longer U4.28 (IO8)
- net OLED-DC: now also U4.16 (IO26); no longer U4.34 (IO22)
- net OLED-MOSI: now also U4.12 (IO32); no longer U4.26 (IO20)
- net OLED-RST: now also U4.17 (IO27); no longer U4.35 (IO21)
- net OLED-SCLK: now also U4.13 (IO33); no longer U4.27 (IO7)
- net R: now also U4.27 (IO7); no longer U4.20 (IO13)
- net TEMP: now also R13.1, U4.18 (IO14); no longer R13.2, U4.24 (IO4)
- no-connect marks 17 -> 16
Other:
- moved on the sheet: R13, R5, R6

Commit message: Resitors
Parts:
- R1: value 10M 1% or 0R -> 100k 1% or 0R
- R2: value 3M 1% or NF -> 30k 1% or NF
Changed lines of the file:
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@@
       (effects (font (size 1.27 1.27)) (justify left))
     )
-    (property "Value" "10M 1% or 0R" (id 1) (at 46.355 144.78 90)
+    (property "Value" "100k 1% or 0R" (id 1) (at 46.355 144.78 90)
       (effects (font (size 1.27 1.27)) (justify left))
     )
@@
       (effects (font (size 1.27 1.27)) (justify right))
     )
-    (property "Value" "3M 1% or NF" (id 1) (at 51.435 145.415 0)
+    (property "Value" "30k 1% or NF" (id 1) (at 51.435 145.415 0)
       (effects (font (size 1.27 1.27)) (justify right))
     )
@@
     )
     (path "/6324f539-5157-429d-ad08-999e5f3ad633"
-      (reference "R1") (unit 1) (value "10M 1% or 0R") (footprint "RevK:R_0603")
+      (reference "R1") (unit 1) (value "100k 1% or 0R") (footprint "RevK:R_0603")
     )
     (path "/e632df6d-ccd6-4691-adc1-89013dd5fd28"
-      (reference "R2") (unit 1) (value "3M 1% or NF") (footprint "RevK:R_0603")
+      (reference "R2") (unit 1) (value "30k 1% or NF") (footprint "RevK:R_0603")
     )
     (path "/00000000-0000-0000-0000-0000604954a7"
