File: KiCad/EnvMon2.kicad_sch (KiCad schematic)
At the start: 37 parts, among them J1 USB-C, J2 DC, J3 TEMP, J4 Shelly, M1 OLED1.5-RGB, SW1 SW_Push, SW2 SW_Push, SW3 SW_Push, U1 LMR16006+FB, U2 SCD41, U3 FT231XQ, U4 ESP32-PICO-MINI-02, U5 QR, U6 VEML3235SL

Commit message: Right angle
Parts:
- U6: value VEML3235SL -> VEML3235SL-RA; footprint RevK:VEML3235SL -> RevK:VEML3235SL-RA
Changed lines of the file:
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@@
       (effects (font (size 1.27 1.27)) (justify left))
     )
-    (property "Value" "VEML3235SL" (id 1) (at 172.085 138.5447 0)
+    (property "Value" "VEML3235SL-RA" (id 1) (at 172.085 138.5447 0)
       (effects (font (size 1.27 1.27)) (justify left))
     )
-    (property "Footprint" "RevK:VEML3235SL" (id 2) (at 164.465 136.525 0)
+    (property "Footprint" "RevK:VEML3235SL-RA" (id 2) (at 164.465 136.525 0)
       (effects (font (size 1.27 1.27)) hide)
     )
@@
     )
     (path "/e1abd673-fcdf-459b-bb90-f108575d9b74"
-      (reference "U6") (unit 1) (value "VEML3235SL") (footprint "RevK:VEML3235SL")
-    )
-  )
+      (reference "U6") (unit 1) (value "VEML3235SL-RA") (footprint "RevK:VEML3235SL-RA")
+    )
+  )

Commit message: Minor tweaks
Parts:
- J1: footprint RevK:USC16-TR-Round -> RevK:USC16-TR
Changed lines of the file:
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@@
     (property "Reference" "J1" (id 0) (at 43.3578 21.1582 0))
     (property "Value" "USB-C" (id 1) (at 43.3578 23.4696 0))
-    (property "Footprint" "RevK:USC16-TR-Round" (id 2) (at 44.45 43.18 0)
+    (property "Footprint" "RevK:USC16-TR" (id 2) (at 44.45 43.18 0)
       (effects (font (size 1.27 1.27)) hide)
     )
@@
     )
     (path "/00000000-0000-0000-0000-0000604764e2"
-      (reference "J1") (unit 1) (value "USB-C") (footprint "RevK:USC16-TR-Round")
+      (reference "J1") (unit 1) (value "USB-C") (footprint "RevK:USC16-TR")
     )
     (path "/05c95e20-b8ce-45a0-abe6-40ea1ba1906f"

Commit message: Library update
Connections:
- net BOOT: now also J4.2 (0); no longer J4.4 (Rx)
- net GND: now also J4.1 (GND); no longer J4.5 (Tx)
- net I: now also J4.4 (Rx); no longer J4.2 (0)
- net O: now also J4.5 (Tx); no longer J4.1 (GND)
Other:
- moved on the sheet: J4
Changed lines of the file:
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@@
     (comment 2 "www.me.uk")
   )
+  (junction (at 160.02 58.42) (diameter 0) (color 0 0 0 0)
+  )
+  (junction (at 129.54 20.32) (diameter 0) (color 0 0 0 0)
+  )
+  (junction (at 58.42 96.52) (diameter 0) (color 0 0 0 0)
+  )
+  (junction (at 43.18 131.445) (diameter 0) (color 0 0 0 0)
+  )
+  (junction (at 226.06 46.99) (diameter 0) (color 0 0 0 0)
+  )
+  (junction (at 193.04 38.1) (diameter 0) (color 0 0 0 0)
+  )
+  (junction (at 114.3 27.94) (diameter 0) (color 0 0 0 0)
+  )
+  (junction (at 74.295 27.94) (diameter 0) (color 0 0 0 0)
+  )
+  (junction (at 226.06 52.07) (diameter 0) (color 0 0 0 0)
+  )
   (junction (at 226.06 41.91) (diameter 0) (color 0 0 0 0)
   )
-  (junction (at 160.02 58.42) (diameter 0) (color 0 0 0 0)
-  )
-  (junction (at 129.54 20.32) (diameter 0) (color 0 0 0 0)
-  )
-  (junction (at 58.42 96.52) (diameter 0) (color 0 0 0 0)
-  )
-  (junction (at 43.18 131.445) (diameter 0) (color 0 0 0 0)
-  )
-  (junction (at 193.04 38.1) (diameter 0) (color 0 0 0 0)
-  )
-  (junction (at 114.3 27.94) (diameter 0) (color 0 0 0 0)
-  )
-  (junction (at 74.295 27.94) (diameter 0) (color 0 0 0 0)
+  (junction (at 132.08 66.04) (diameter 0) (color 0 0 0 0)
+  )
+  (junction (at 43.18 127) (diameter 0) (color 0 0 0 0)
+  )
+  (junction (at 49.53 141.605) (diameter 0) (color 0 0 0 0)
+  )
+  (junction (at 38.735 139.065) (diameter 0) (color 0 0 0 0)
+  )
+  (junction (at 66.04 107.95) (diameter 0) (color 0 0 0 0)
+  )
+  (junction (at 66.04 33.02) (diameter 0) (color 0 0 0 0)
+  )
+  (junction (at 40.64 66.04) (diameter 0) (color 0 0 0 0)
+  )
+  (junction (at 226.06 49.53) (diameter 0) (color 0 0 0 0)
   )
   (junction (at 226.06 44.45) (diameter 0) (color 0 0 0 0)
-  )
-  (junction (at 132.08 66.04) (diameter 0) (color 0 0 0 0)
-  )
-  (junction (at 226.06 52.07) (diameter 0) (color 0 0 0 0)
-  )
-  (junction (at 43.18 127) (diameter 0) (color 0 0 0 0)
-  )
-  (junction (at 49.53 141.605) (diameter 0) (color 0 0 0 0)
-  )
-  (junction (at 38.735 139.065) (diameter 0) (color 0 0 0 0)
-  )
-  (junction (at 66.04 107.95) (diameter 0) (color 0 0 0 0)
-  )
-  (junction (at 226.06 46.99) (diameter 0) (color 0 0 0 0)
-  )
-  (junction (at 66.04 33.02) (diameter 0) (color 0 0 0 0)
-  )
-  (junction (at 40.64 66.04) (diameter 0) (color 0 0 0 0)
-  )
-  (junction (at 226.06 49.53) (diameter 0) (color 0 0 0 0)
   )
   (junction (at 79.375 27.94) (diameter 0) (color 0 0 0 0)
@@
   (no_connect (at 195.58 48.26))
   (no_connect (at 195.58 73.66))
+  (wire (pts (xy 55.88 33.02) (xy 58.42 33.02))
+    (stroke (width 0) (type default) (color 0 0 0 0))
+  )
+  (wire (pts (xy 55.88 27.94) (xy 74.295 27.94))
+    (stroke (width 0) (type default) (color 0 0 0 0))
+  )
+  (wire (pts (xy 66.04 33.02) (xy 66.04 35.56))
+    (stroke (width 0) (type default) (color 0 0 0 0))
+  )
+  (wire (pts (xy 38.735 136.525) (xy 49.53 136.525))
+    (stroke (width 0) (type default) (color 0 0 0 0))
+  )
+  (wire (pts (xy 106.68 27.94) (xy 106.68 43.18))
+    (stroke (width 0) (type default) (color 0 0 0 0))
+  )
+  (wire (pts (xy 79.375 27.94) (xy 79.375 33.02))
+    (stroke (width 0) (type default) (color 0 0 0 0))
+  )
+  (wire (pts (xy 55.88 45.72) (xy 58.42 45.72))
+    (stroke (width 0) (type default) (color 0 0 0 0))
+  )
+  (wire (pts (xy 193.04 38.1) (xy 195.58 38.1))
+    (stroke (width 0) (type default) (color 0 0 0 0))
+  )
+  (wire (pts (xy 38.735 139.065) (xy 49.53 139.065))
+    (stroke (width 0) (type default) (color 0 0 0 0))
+  )
+  (wire (pts (xy 43.18 127) (xy 50.165 127))
+    (stroke (width 0) (type default) (color 0 0 0 0))
+  )
+  (wire (pts (xy 114.3 27.94) (xy 106.68 27.94))
+    (stroke (width 0) (type default) (color 0 0 0 0))
+  )
+  (wire (pts (xy 33.02 66.04) (xy 40.64 66.04))
+    (stroke (width 0) (type default) (color 0 0 0 0))
+  )
+  (wire (pts (xy 46.355 141.605) (xy 49.53 141.605))
+    (stroke (width 0) (type default) (color 0 0 0 0))
+  )
+  (wire (pts (xy 226.06 41.91) (xy 229.235 41.91))
+    (stroke (width 0) (type default) (color 0 0 0 0))
+  )
+  (wire (pts (xy 106.68 43.18) (xy 114.3 43.18))
+    (stroke (width 0) (type default) (color 0 0 0 0))
+  )
+  (wire (pts (xy 58.42 96.52) (xy 58.42 99.06))
+    (stroke (width 0) (type default) (color 0 0 0 0))
+  )
+  (wire (pts (xy 43.18 123.825) (xy 43.18 127))
+    (stroke (width 0) (type default) (color 0 0 0 0))
+  )
+  (wire (pts (xy 48.26 123.825) (xy 43.18 123.825))
+    (stroke (width 0) (type default) (color 0 0 0 0))
+  )
+  (wire (pts (xy 55.88 35.56) (xy 58.42 35.56))
+    (stroke (width 0) (type default) (color 0 0 0 0))
+  )
+  (wire (pts (xy 226.06 52.07) (xy 229.235 52.07))
+    (stroke (width 0) (type default) (color 0 0 0 0))
+  )
+  (wire (pts (xy 226.06 44.45) (xy 229.235 44.45))
+    (stroke (width 0) (type default) (color 0 0 0 0))
+  )
+  (wire (pts (xy 74.295 27.94) (xy 79.375 27.94))
+    (stroke (width 0) (type default) (color 0 0 0 0))
+  )
+  (wire (pts (xy 43.18 127) (xy 43.18 131.445))
+    (stroke (width 0) (type default) (color 0 0 0 0))
+  )
+  (wire (pts (xy 114.3 20.32) (xy 129.54 20.32))
+    (stroke (width 0) (type default) (color 0 0 0 0))
+  )
+  (wire (pts (xy 66.04 107.95) (xy 68.58 107.95))
+    (stroke (width 0) (type default) (color 0 0 0 0))
+  )
+  (wire (pts (xy 226.06 49.53) (xy 229.235 49.53))
+    (stroke (width 0) (type default) (color 0 0 0 0))
+  )
+  (wire (pts (xy 55.88 43.18) (xy 58.42 43.18))
+    (stroke (width 0) (type default) (color 0 0 0 0))
+  )
+  (wire (pts (xy 114.3 27.94) (xy 114.3 20.32))
+    (stroke (width 0) (type default) (color 0 0 0 0))
+  )
   (wire (pts (xy 226.06 46.99) (xy 229.235 46.99))
-    (stroke (width 0) (type default) (color 0 0 0 0))
-  )
-  (wire (pts (xy 55.88 33.02) (xy 58.42 33.02))
-    (stroke (width 0) (type default) (color 0 0 0 0))
-  )
-  (wire (pts (xy 55.88 27.94) (xy 74.295 27.94))
-    (stroke (width 0) (type default) (color 0 0 0 0))
-  )
-  (wire (pts (xy 66.04 33.02) (xy 66.04 35.56))
-    (stroke (width 0) (type default) (color 0 0 0 0))
-  )
-  (wire (pts (xy 38.735 136.525) (xy 49.53 136.525))
-    (stroke (width 0) (type default) (color 0 0 0 0))
-  )
-  (wire (pts (xy 106.68 27.94) (xy 106.68 43.18))
-    (stroke (width 0) (type default) (color 0 0 0 0))
-  )
-  (wire (pts (xy 79.375 27.94) (xy 79.375 33.02))
-    (stroke (width 0) (type default) (color 0 0 0 0))
-  )
-  (wire (pts (xy 55.88 45.72) (xy 58.42 45.72))
-    (stroke (width 0) (type default) (color 0 0 0 0))
-  )
-  (wire (pts (xy 193.04 38.1) (xy 195.58 38.1))
-    (stroke (width 0) (type default) (color 0 0 0 0))
-  )
-  (wire (pts (xy 38.735 139.065) (xy 49.53 139.065))
-    (stroke (width 0) (type default) (color 0 0 0 0))
-  )
-  (wire (pts (xy 43.18 127) (xy 50.165 127))
-    (stroke (width 0) (type default) (color 0 0 0 0))
-  )
-  (wire (pts (xy 114.3 27.94) (xy 106.68 27.94))
-    (stroke (width 0) (type default) (color 0 0 0 0))
-  )
-  (wire (pts (xy 33.02 66.04) (xy 40.64 66.04))
-    (stroke (width 0) (type default) (color 0 0 0 0))
-  )
-  (wire (pts (xy 46.355 141.605) (xy 49.53 141.605))
-    (stroke (width 0) (type default) (color 0 0 0 0))
-  )
-  (wire (pts (xy 226.06 41.91) (xy 229.235 41.91))
-    (stroke (width 0) (type default) (color 0 0 0 0))
-  )
-  (wire (pts (xy 106.68 43.18) (xy 114.3 43.18))
-    (stroke (width 0) (type default) (color 0 0 0 0))
-  )
-  (wire (pts (xy 58.42 96.52) (xy 58.42 99.06))
-    (stroke (width 0) (type default) (color 0 0 0 0))
-  )
-  (wire (pts (xy 43.18 123.825) (xy 43.18 127))
-    (stroke (width 0) (type default) (color 0 0 0 0))
-  )
-  (wire (pts (xy 48.26 123.825) (xy 43.18 123.825))
-    (stroke (width 0) (type default) (color 0 0 0 0))
-  )
-  (wire (pts (xy 55.88 35.56) (xy 58.42 35.56))
-    (stroke (width 0) (type default) (color 0 0 0 0))
-  )
-  (wire (pts (xy 226.06 52.07) (xy 229.235 52.07))
-    (stroke (width 0) (type default) (color 0 0 0 0))
-  )
-  (wire (pts (xy 226.06 44.45) (xy 229.235 44.45))
-    (stroke (width 0) (type default) (color 0 0 0 0))
-  )
-  (wire (pts (xy 74.295 27.94) (xy 79.375 27.94))
-    (stroke (width 0) (type default) (color 0 0 0 0))
-  )
-  (wire (pts (xy 43.18 127) (xy 43.18 131.445))
-    (stroke (width 0) (type default) (color 0 0 0 0))
-  )
-  (wire (pts (xy 114.3 20.32) (xy 129.54 20.32))
-    (stroke (width 0) (type default) (color 0 0 0 0))
-  )
-  (wire (pts (xy 66.04 107.95) (xy 68.58 107.95))
-    (stroke (width 0) (type default) (color 0 0 0 0))
-  )
-  (wire (pts (xy 226.06 49.53) (xy 229.235 49.53))
-    (stroke (width 0) (type default) (color 0 0 0 0))
-  )
-  (wire (pts (xy 55.88 43.18) (xy 58.42 43.18))
-    (stroke (width 0) (type default) (color 0 0 0 0))
-  )
-  (wire (pts (xy 114.3 27.94) (xy 114.3 20.32))
     (stroke (width 0) (type default) (color 0 0 0 0))
   )
@@
     (pin "1")
   )
-  (symbol (lib_id "RevK:Shelly") (at 226.06 46.99 0) (unit 1)
+  (symbol (lib_id "RevK:Shelly") (at 226.06 46.99 180) (unit 1)
     (in_bom no) (on_board yes) (fields_autoplaced)
-    (property "Reference" "J4" (id 0) (at 226.06 37.626 0))
-    (property "Value" "Shelly" (id 1) (at 226.06 40.1629 0))
-    (property "Footprint" "RevK:Shelly" (id 2) (at 228.6 55.245 0)
-      (effects (font (size 1.27 1.27)) hide)
-    )
-    (property "Datasheet" "" (id 3) (at 228.6 55.245 0)
-      (effects (font (size 1.27 1.27)) hide)
-    )
+    (property "Reference" "J4" (id 0) (at 227.4062 46.1553 0)
+      (effects (font (size 1.27 1.27)) (justify right))
+    )
+    (property "Value" "Shelly" (id 1) (at 227.4062 48.6922 0)
+      (effects (font (size 1.27 1.27)) (justify right))
+    )
+    (property "Footprint" "RevK:Shelly" (id 2) (at 223.52 38.735 0)
+      (effects (font (size 1.27 1.27)) hide)
+    )
+    (property "Datasheet" "" (id 3) (at 223.52 38.735 0)
+      (effects (font (size 1.27 1.27)) hide)
+    )
