File: PCB/EnvMon2/EnvMon2.kicad_pcb (KiCad board)
At the start: 2 copper layers, 57.5 x 37 mm, 38 parts, among them J1 USB-C, J2 DC, J3 TEMP, J4 Shelly, M1 OLED1.5-RGB, SW1 SW_Push, SW2 SW_Push, SW3 SW_Push, U1 LMR16006+FB, U2 SCD41, U3 FT231XQ, U4 ESP32-PICO-MINI-02, U5 QR, U6 VEML3235SL-RA

Commit message: Production files, not finished
Other:
- rule pad_to_mask_clearance: 0.01 -> 0
Changed lines of the file:
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@@
       (dielectric_constraints no)
     )
-    (pad_to_mask_clearance 0.01)
+    (pad_to_mask_clearance 0)
     (pad_to_paste_clearance_ratio -0.02)
     (pcbplotparams

Commit message: Library update
Parts:
- removed ?: , RevK:PasteEnvMon2
- C1: footprint RevK:C_0603_ -> RevK:Hidden
- C2, C3: footprint RevK:C_0805_ -> RevK:Hidden
- D1: footprint RevK:D_1206_ -> RevK:Hidden
- D3: value RGB -> LED_BARG; footprint RevK:LED-RGB-1.6x1.6 -> RevK:MHS190RGBCT
- L1: footprint RevK:L_4x4_ -> RevK:Hidden
- R1: value 100k 1% or 0R -> 100k 1%
- R2: value 30k 1% or NF -> 30k 1%
- U1: value LMR16006+FB -> LMR16006XDDCR; footprint RevK:RegulatorBlockFB -> RevK:SOT-23-Thin-6-Reg
- U3: footprint RevK:QFN-20-1EP_4x4mm_P0.5mm_EP2.5x2.5mm -> RevK:JLC-QFN-20-1EP_4x4mm_P0.5mm_EP2.5x2.5m
- moved J1 4.40 mm to (122.2, 95.6)
- moved R8 3.54 mm to (138.0, 69.6), turned to -90 degrees
- moved R9 2.51 mm to (135.8, 69.6), turned to -90 degrees
- moved R7 1.00 mm to (136.9, 69.6), turned to -90 degrees
- moved D3 0.44 mm to (136.9, 64.2), turned to 0 degrees
- turned U1 to 0 degrees
- turned U3 to -90 degrees
Connections:
- D3 pad 1: +3V3 -> Net-(D3-Pad1)
- D3 pad 2: Net-(D3-Pad2) -> +3.3V
- J3 pad 3: +3V3 -> +3.3V
- J4 pad 3: +3V3 -> +3.3V
- M1 pad 1: +3V3 -> +3.3V
- R1 pad 1: +3V3 -> +3.3V
- R12 pad 1: +3V3 -> +3.3V
- R13 pad 2: +3V3 -> +3.3V
- R7 pad 1: Net-(D3-Pad2) -> Net-(D3-Pad3)
- R8 pad 1: Net-(D3-Pad3) -> Net-(D3-Pad4)
- R9 pad 1: Net-(D3-Pad4) -> Net-(D3-Pad1)
- U1 pad 4: +3V3 -> +3.3V
- U2 pad 19: +3V3 -> +3.3V
- U2 pad 7: +3V3 -> +3.3V
- U3 pad 10: +3V3 -> +3.3V
- U3 pad 11: +3V3 -> +3.3V
- U3 pad 12: +3V3 -> +3.3V
- U3 pad 20: +3V3 -> +3.3V
- U4 pad 27: R -> G
- U4 pad 28: B -> R
- U4 pad 3: +3V3 -> +3.3V
- U4 pad 33: G -> B
- U6 pad 1: +3V3 -> +3.3V
Routing:
- net +3V3: track 178.2 -> 0.00 mm, vias 3 -> 0
- net +3.3V: track 0.00 -> 174.8 mm, vias 0 -> 3
- net B: track 14.0 -> 8.27 mm
- net Net-(D3-Pad2): track 5.48 -> 0.00 mm
- net Net-(D3-Pad1): track 0.00 -> 4.83 mm
- net Net-(D3-Pad3): track 1.12 -> 4.66 mm
- net G: track 12.0 -> 14.3 mm
- net Net-(D3-Pad4): track 3.29 -> 4.83 mm
- net R: track 13.5 -> 12.2 mm
- net GND: track 20.6 -> 19.8 mm
- net OLED-CS: track 20.8 -> 20.1 mm
- net BOOT: track 31.7 -> 31.1 mm

Commit message: Revised production files
Parts:
- C1: footprint RevK:Hidden -> RevK:C_0603_
- C2, C3: footprint RevK:Hidden -> RevK:C_0805_
- D1: footprint RevK:Hidden -> RevK:D_1206_
- L1: footprint RevK:Hidden -> RevK:L_4x4_
- U3: footprint RevK:JLC-QFN-20-1EP_4x4mm_P0.5mm_EP2.5x2.5m -> RevK:QFN-20-1EP_4x4mm_P0.5mm_EP2.5x2.5mm
- U6: value VEML3235SL-RA -> VEML3235SL_RA
- turned U3 to 0 degrees

Commit message: LED pin silkscreen fix
Other:
- board text added: "LED: 8/7/19"
- board text removed: "LED: 7/19/8"
Changed lines of the file:
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@@
     (effects (font (size 0.75 0.75) (thickness 0.15)) (justify mirror))
   )
-  (gr_text "LED: 7/19/8" (at 139.5 69.5) (layer "B.SilkS")
+  (gr_text "LED: 8/7/19" (at 139.5 69.5) (layer "B.SilkS")
     (effects (font (size 0.75 0.75) (thickness 0.15)) (justify mirror))
   )

Commit message: Production file update
Parts:
- turned U1 to 90 degrees
Connections:
- U1 pad 1: DC -> unconnected-(U1-Pad1)
- U1 pad 2: DC -> GND
- U1 pad 3: GND -> Net-(R1-Pad2)
- U1 pad 4: +3.3V -> DC
- U1 pad 5: Net-(R1-Pad2) -> DC

Commit message: Resistor update for LED
Parts:
- R7: value 680R -> 300R
- R8: value 2K -> 1K
- R9: value 220R -> 100R
Changed lines of the file:
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@@
       (effects (font (size 0.5 0.5) (thickness 0.08)))
     )
-    (fp_text value "680R" (at 0 0 -270) (layer "F.Fab")
+    (fp_text value "300R" (at 0 0 -270) (layer "F.Fab")
       (effects (font (size 0.4 0.4) (thickness 0.08)))
     )
@@
       (effects (font (size 0.5 0.5) (thickness 0.08)))
     )
-    (fp_text value "2K" (at 0 0 -270) (layer "F.Fab")
+    (fp_text value "1K" (at 0 0 -270) (layer "F.Fab")
       (effects (font (size 0.4 0.4) (thickness 0.08)))
     )
@@
       (effects (font (size 0.5 0.5) (thickness 0.08)))
     )
-    (fp_text value "220R" (at 0 0 -270) (layer "F.Fab")
+    (fp_text value "100R" (at 0 0 -270) (layer "F.Fab")
       (effects (font (size 0.4 0.4) (thickness 0.08)))
     )

Commit message: Extra diode
Parts:
- added D4: D, RevK:D_1206, F.Cu at (139.2, 91.4)
Connections:
- J2 pad 2: DC -> Net-(J2-Pad2)
Routing:
- net Net-(J2-Pad2): track 0.00 -> 3.69 mm
- net DC: track 11.9 -> 10.5 mm
Changed lines of the file:
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@@
     )
   )
-  (property "DATE" "2023-01-11")
+  (property "DATE" "2023-01-20")
   (net 0 "")
   (net 1 "VBUS")
@@
   (net 65 "unconnected-(U1-Pad1)")
   (net 66 "unconnected-(U1-Pad6)")
+  (net 67 "Net-(J2-Pad2)")
   (footprint "Button_Switch_THT:SW_PUSH_6mm_H13mm" (layer "F.Cu")
     (at 89.25 65.25)
@@
     (property "Sheetfile" "EnvMon2.kicad_sch")
     (property "Sheetname" "")
-    (property "exclude_from_bom" "")
-    (attr through_hole exclude_from_bom)
+    (attr through_hole)
     (fp_text reference "J3" (at 0 6) (layer "F.SilkS") hide
       (effects (font (size 1 1) (thickness 0.15)))
@@
       (scale (xyz 1 1 1))
       (rotate (xyz 0 0 180))
+    )
+  )
+  (footprint "RevK:D_1206" (layer "F.Cu")
+    (at 139.2 91.4 180)
+    (descr "Diode SMD 1206 (3216 Metric), square (rectangular) end terminal, IPC_7351 nominal, (Body size source: http://www.tortai-tech.com/upload/download/2011102023233369053.pdf), generated with kicad-footprint-generator")
+    (tags "diode")
+    (property "LCSC Part #" "C143805")
+    (property "Sheetfile" "EnvMon2.kicad_sch")
+    (property "Sheetname" "")
+    (attr smd)
+    (fp_text reference "D4" (at 0 -1.82) (layer "F.SilkS") hide
+      (effects (font (size 1 1) (thickness 0.15)))
+    )
+    (fp_text value "D" (at 0 1.82) (layer "F.Fab")
+      (effects (font (size 1 1) (thickness 0.15)))
+    )
+    (fp_text user "${REFERENCE}" (at 0 0) (layer "F.Fab")
+      (effects (font (size 0.8 0.8) (thickness 0.12)))
+    )
+    (fp_line (start -0.5 -0.75) (end -0.5 0.75) (layer "F.SilkS") (width 0.12))
+    (fp_line (start -2.28 -1.12) (end 2.28 -1.12) (layer "F.CrtYd") (width 0.05))
+    (fp_line (start -2.28 1.12) (end -2.28 -1.12) (layer "F.CrtYd") (width 0.05))
+    (fp_line (start 2.28 1.12) (end -2.28 1.12) (layer "F.CrtYd") (width 0.05))
+    (fp_line (start 2.28 -1.12) (end 2.28 1.12) (layer "F.CrtYd") (width 0.05))
+    (fp_line (start -1.2 -0.8) (end -1.6 -0.4) (layer "F.Fab") (width 0.1))
+    (fp_line (start 1.6 -0.8) (end -1.2 -0.8) (layer "F.Fab") (width 0.1))
+    (fp_line (start -1.6 -0.4) (end -1.6 0.8) (layer "F.Fab") (width 0.1))
+    (fp_line (start -1.6 0.8) (end 1.6 0.8) (layer "F.Fab") (width 0.1))
+    (fp_line (start 1.6 0.8) (end 1.6 -0.8) (layer "F.Fab") (width 0.1))
+    (pad "1" smd roundrect (at -1.4 0 180) (size 1.25 1.75) (layers "F.Cu" "F.Paste" "F.Mask") (roundrect_rratio 0.2)
+      (net 30 "DC") (pinfunction "K") (pintype "passive"))
+    (pad "2" smd roundrect (at 1.4 0 180) (size 1.25 1.75) (layers "F.Cu" "F.Paste" "F.Mask") (roundrect_rratio 0.2)
+      (net 67 "Net-(J2-Pad2)") (pinfunction "A") (pintype "passive"))
+    (model "${KICAD6_3DMODEL_DIR}/Diode_SMD.3dshapes/D_1206_3216Metric.wrl"
+      (offset (xyz 0 0 0))
+      (scale (xyz 1 1 1))
+      (rotate (xyz 0 0 0))
     )
   )
@@
       (net 11 "GND") (pinfunction "GND") (pintype "power_in"))
     (pad "2" thru_hole oval (at 1.25 0) (size 1.7 1.85) (drill 0.85) (layers *.Cu *.Mask)
-      (net 30 "DC") (pinfunction "DC") (pintype "power_out"))
+      (net 67 "Net-(J2-Pad2)") (pinfunction "DC") (pintype "power_out"))
     (model "/Users/adrian/Documents/KiCad/3D/22057025.stp"
       (offset (xyz 0 -3.6 2.5))
@@
   (arc (start 134.63175 71.59325) (mid 135.457827 71.251077) (end 135.8 70.425) (width 0.25) (layer "F.Cu") (net 29))
   (segment (start 136 85.85) (end 135.224264 85.074264) (width 0.5) (layer "F.Cu") (net 30))
-  (segment (start 136.35 90.85) (end 134.25 90.85) (width 0.5) (layer "F.Cu") (net 30))
-  (segment (start 137.75 87.6) (end 137.75 89.45) (width 0.5) (layer "F.Cu") (net 30))
   (segment (start 133.55 84.15) (end 133.55 83.2) (width 0.25) (layer "F.Cu") (net 30))
-  (arc (start 137.75 89.45) (mid 137.339949 90.439949) (end 136.35 90.85) (width 0.5) (layer "F.Cu") (net 30))
-  (arc (start 136 85.85) (mid 137.237437 86.362563) (end 137.75 87.6) (width 0.5) (layer "F.Cu") (net 30))
+  (segment (start 136 85.85) (end 139.928248 89.778248) (width 0.5) (layer "F.Cu") (net 30))
+  (arc (start 139.928248 89.778248) (mid 140.425417 90.522314) (end 140.6 91.4) (width 0.5) (layer "F.Cu") (net 30))
   (arc (start 135.224264 85.074264) (mid 134.910263 84.604328) (end 134.8 84.05) (width 0.5) (layer "F.Cu") (net 30))
   (segment (start 137.125 64.175) (end 137.125 68.231802) (width 0.25) (layer "F.Cu") (net 31))
@@
   (arc (start 124.55 86.75) (mid 124.196447 86.896447) (end 124.05 87.25) (width 0.25) (layer "B.Cu") (net 64))
   (arc (start 129.5 86.75) (mid 131.409188 85.959188) (end 132.2 84.05) (width 0.25) (layer "B.Cu") (net 64))
+  (segment (start 134.25 90.85) (end 136.472183 90.85) (width 0.5) (layer "F.Cu") (net 67))
+  (arc (start 136.472183 90.85) (mid 137.190792 90.992941) (end 137.8 91.4) (width 0.5) (layer "F.Cu") (net 67))
   (zone (net 11) (net_name "GND") (layers F&B.Cu) (hatch edge 0.508)
     (connect_pads thru_hole_only (clearance 0.25))
