File: PCB/EnvMon2/EnvMon.kicad_pcb (KiCad board)
At the start: 2 copper layers, 57.5 x 37 mm, 37 parts, among them J1 USB-C, J2 DC, J3 TEMP, J5 Shelly, M1 OLED1.5-RGB, SW1 SW_Push, SW2 SW_Push, SW3 SW_Push, U1 ESP32-S3-MINI-1, U2 SCD41, U5 QR, U6 MD8942, U7 SHT40, U8 VEML6040

Commit message: Pretty tracks
Parts:
- removed D4: D, RevK:D_1206
- added D3: D, RevK:D_SOD-123, F.Cu at (126.5, 90.3)
- D2: footprint RevK:D_1206 -> RevK:D_SOD-123
- moved C5 1.95 mm to (140.6, 69.4), turned to 180 degrees
- moved D2 1.90 mm to (128.4, 90.3)
- moved Logo2 1.51 mm to (108.5, 75.7)
- moved R1 0.70 mm to (136.4, 66.3)
- moved D1 0.70 mm to (136.4, 64.5)
- moved R17 0.70 mm to (135.7, 66.3)
- moved R2 0.70 mm to (137.2, 66.3)
- moved U7 0.56 mm to (140.6, 70.8), turned to 90 degrees
Connections:
- J1 pad A4: Net-(D2-A) -> Net-(D3-A)
- J1 pad A9: Net-(D2-A) -> Net-(D3-A)
- J1 pad B4: Net-(D2-A) -> Net-(D3-A)
- J1 pad B9: Net-(D2-A) -> Net-(D3-A)
- J2 pad 2: Net-(D4-A) -> Net-(D2-A)
Routing:
- net OLED-MOSI: track 12.3 -> 25.2 mm
- net BUTTON3: track 27.0 -> 36.9 mm
- net Net-(D3-A): track 0.00 -> 9.26 mm
- net SDA: track 88.6 -> 95.7 mm
- net Net-(D4-A): track 6.37 -> 0.00 mm
- net SCL: track 91.0 -> 95.0 mm
- net +3.3V: track 150.6 -> 154.4 mm
- net Net-(J5-Tx): track 7.15 -> 10.3 mm
- net Net-(D2-A): track 9.62 -> 6.57 mm
- net OLED-DC: track 15.0 -> 13.7 mm
- net BUTTON1: track 31.1 -> 29.9 mm
- net G: track 14.4 -> 13.7 mm
- net R: track 13.2 -> 12.6 mm
- net B: track 12.1 -> 11.4 mm
- net OLED-RST: track 15.7 -> 15.1 mm
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Other:
- outline, holes or cut-outs redrawn
