File: PCB/USBC/USBC.kicad_pcb (KiCad board)
At the start: 2 copper layers, 70 x 70 mm, 27 parts, among them J1 USB-C-Plug-V, J2 Shelly, J3 USB-PROG, U2 ESP32-S3-MINI-1, U3 SCD41, U5 MD8942

Commit message: Tidy
Parts:
- U3: value SCD41 -> SCD41-D-R1
Other:
- board text added: "www.me.uk"
- board text removed: "BA"

Commit message: Tidy
Other:
- board text removed: "+"
Changed lines of the file:
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@@
-    )
-  )
-  (gr_text "+" (at 103.1 105.7) (layer "B.SilkS")
-    (effects (font (face "OCR-B") (size 1.2 1.2) (thickness 0.15)) (justify mirror))
-    (render_cache "+" 0
-      (polygon
-        (pts
-          (xy 103.517655 105.552612)          (xy 103.516661 105.565187)          (xy 103.512435 105.58002)          (xy 103.505238 105.592598)
-          (xy 103.495443 105.602872)          (xy 103.483425 105.610796)          (xy 103.469558 105.616321)          (xy 103.454217 105.619398)
-          (xy 103.441969 105.620071)          (xy 103.433537 105.61973)          (xy 103.164773 105.61973)          (xy 103.164773 105.937441)
-          (xy 103.164199 105.950345)          (xy 103.162472 105.962591)          (xy 103.15958 105.974044)          (xy 103.153897 105.987852)
-          (xy 103.146102 105.999699)          (xy 103.136171 106.009269)          (xy 103.124081 106.016246)          (xy 103.109807 106.020314)
-          (xy 103.097655 106.021265)          (xy 103.085495 106.020272)          (xy 103.071192 106.016049)          (xy 103.059058 106.00886)
-          (xy 103.049075 105.999084)          (xy 103.041226 105.987097)          (xy 103.035493 105.973277)          (xy 103.031859 105.958004)
-          (xy 103.030502 105.945821)          (xy 103.030244 105.937441)          (xy 103.030244 105.61973)          (xy 102.761479 105.61973)
-          (xy 102.748913 105.619157)          (xy 102.736874 105.617429)          (xy 102.721907 105.613313)          (xy 102.708518 105.607104)
-          (xy 102.697076 105.598778)          (xy 102.687946 105.588309)          (xy 102.681497 105.575676)          (xy 102.678097 105.560852)
-          (xy 102.677655 105.552612)          (xy 102.678641 105.540375)          (xy 102.682838 105.525788)          (xy 102.689992 105.513266)
-          (xy 102.699734 105.502903)          (xy 102.711697 105.494798)          (xy 102.725515 105.489045)          (xy 102.740819 105.485741)
-          (xy 102.753051 105.484928)          (xy 102.761479 105.485201)          (xy 103.030244 105.485201)          (xy 103.030244 105.169542)
-          (xy 103.030782 105.156969)          (xy 103.032421 105.144909)          (xy 103.036374 105.129902)          (xy 103.042421 105.116462)
-          (xy 103.05064 105.104965)          (xy 103.06111 105.095784)          (xy 103.073911 105.089294)          (xy 103.089121 105.08587)
-          (xy 103.097655 105.085424)          (xy 103.110146 105.086376)          (xy 103.124668 105.090447)          (xy 103.136822 105.097432)
-          (xy 103.146683 105.107021)          (xy 103.154327 105.118899)          (xy 103.15983 105.132755)          (xy 103.162597 105.144256)
-          (xy 103.164234 105.156563)          (xy 103.164773 105.169542)          (xy 103.164773 105.485201)          (xy 103.433537 105.485201)
-          (xy 103.44611 105.48574)          (xy 103.45817 105.487379)          (xy 103.473177 105.491332)          (xy 103.486617 105.497378)
-          (xy 103.498115 105.505597)          (xy 103.507295 105.516068)          (xy 103.513785 105.528869)          (xy 103.517209 105.544079)
-        )
-      )
     )
   )

Commit message: neater
Parts:
- moved V1 25.6 mm to (75.7, 99.8), turned to 90 degrees
- moved R2 22.8 mm to (113.2, 93.8), turned to 180 degrees
- moved C7 22.1 mm to (92.4, 99.1), turned to 90 degrees
- moved J1 21.8 mm to (113.2, 99.3)
- moved R10 21.7 mm to (93.1, 102.3), turned to 180 degrees
- moved U3 21.5 mm to (105.7, 99.3)
- moved J2 21.3 mm to (80.2, 99.3), turned to -90 degrees
- moved C10 21.1 mm to (94.2, 103.9), turned to 0 degrees
- moved L2 18.3 mm to (94.9, 95.8), turned to 180 degrees
- moved R9 18.3 mm to (94.9, 102.3), turned to 180 degrees
- moved D3 18.1 mm to (99.4, 101.8), turned to 135 degrees
- moved U2 17.5 mm to (83.7, 99.3), turned to 90 degrees
- moved U5 17.5 mm to (94.9, 100.4), turned to 180 degrees
- moved V2 17.3 mm to (115.7, 99.8), turned to -90 degrees
- moved C5 17.2 mm to (99.4, 100.5), turned to 0 degrees
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Connections:
- U2 pad 13: SDA -> unconnected-(U2-GPIO9-Pad13)
- U2 pad 14: SCL -> unconnected-(U2-GPIO10-Pad14)
- U2 pad 15: LED -> unconnected-(U2-GPIO11-Pad15)
- U2 pad 16: unconnected-(U2-GPIO12-Pad16) -> SDA
- U2 pad 17: GND -> SCL
- U2 pad 29: unconnected-(U2-GPIO34-Pad29) -> LED
Routing:
- net D+: track 17.1 -> 40.2 mm
- net D-: track 15.0 -> 32.1 mm
- net +3.3V: track 68.5 -> 53.0 mm, vias 3 -> 1
- net Net-(U2-EN): track 3.33 -> 17.4 mm, vias 0 -> 2
- net VBUS: track 61.9 -> 48.6 mm, vias 2 -> 1
- net SDA: track 7.91 -> 18.3 mm
- net GND: track 0.00 -> 8.88 mm, vias 22 -> 23
- net SCL: track 9.44 -> 17.8 mm
- net LED: track 7.74 -> 11.9 mm, vias 0 -> 2
- net Net-(J1-CC): track 7.56 -> 6.43 mm
