File: PCB/USBC/USBC.kicad_pcb (KiCad board)
At the start: 2 copper layers, 70 x 70 mm, 27 parts, among them J1 USB-C-Plug-V, J2 Shelly, J3 USB-PROG, U2 ESP32-S3-MINI-1, U3 SCD41-D-R1, U5 MD8942

Commit message: Tidy
Parts:
- moved R2 5.50 mm to (107.7, 93.7)
Routing:
- net Net-(J1-CC): track 6.43 -> 8.09 mm

Commit message: Tidy
Parts:
- moved R2 12.8 mm to (99.4, 103.5)
- turned J1 to -90 degrees
Routing:
- net Net-(J1-CC): track 8.09 -> 13.6 mm
- net D+: track 40.2 -> 41.1 mm
- net GND: vias 23 -> 27

Commit message: Clear defaults and fix ilk
Other:
- board text added: "SDA:12 SCL:13 RGB:34"
- board text removed: "SDA:9 SCL:10 RGB:11"
