File: PCB/USBC/USBC.kicad_pcb (KiCad board)
At the start: 2 copper layers, 70 x 70 mm, 32 parts, among them J1 USB-C-Plug-V, J2 Shelly, J3 USB-PROG, U2 ESP32-S3-MINI-1, U3 SCD41-D-R1, U5 MD8942

Commit message: Tidy
Parts:
- moved D4 2.30 mm to (112.0, 101.4)
- moved D5 2.30 mm to (112.0, 99.3)
- moved D6 2.30 mm to (112.0, 97.2)
Routing:
- net D+: track 44.4 -> 41.2 mm
- net Net-(D3-O): track 17.2 -> 14.9 mm
- net VBUS: track 65.9 -> 68.0 mm

Commit message: Tody
Other:
- board text added: "Unplugging"
- board text added: "Use care"

Commit message: New plugs
Parts:
- C6: value 10uF 50V -> 10uF 35V

Commit message: Tidy
Parts:
- removed J2: Shelly, RevK:Shelly
- removed J3: USB-PROG, RevK:USB-PROG
- added REF**: Shadow, RevK:Shadow, F.Cu at (100.0, 100.0)
Connections:
- U2 pad 39: Net-(J2-Tx) -> unconnected-(U2-GPIO43-Pad39)
- U2 pad 4: Net-(J2-0) -> unconnected-(U2-GPIO0-Pad4)
- U2 pad 40: Net-(J2-Rx) -> unconnected-(U2-GPIO44-Pad40)
Routing:
- net Net-(J2-Rx): track 6.70 -> 0.00 mm
- net VBUS: track 68.0 -> 61.8 mm
- net Net-(J2-0): track 5.18 -> 0.00 mm
- net GND: track 8.88 -> 4.10 mm, vias 30 -> 26
- net Net-(J2-Tx): track 3.49 -> 0.00 mm
- net D-: track 32.1 -> 34.7 mm, vias 0 -> 1
- net Net-(D3-O): track 14.9 -> 16.1 mm
- net SDA: track 18.3 -> 19.3 mm
- net LED: track 12.4 -> 13.1 mm
- net D+: track 41.2 -> 41.6 mm, vias 2 -> 3
- net +3.3V: vias 1 -> 2
Other:
- board text added: "5060634238120"
- board text added: "Made in China for Andrews&Arnold Ltd"
- board text added: "Take care"
- board text removed: "Use care"
