File: PCB/USBC/USBC.kicad_sch (KiCad schematic)
At the start: 29 parts, among them J1 USB-C-Plug-V, J2 Shelly, J3 USB-PROG, J4 Conn_01x03_Socket, U2 ESP32-S3-MINI-1, U5 MD8942, U8 VEML6040

Commit message: New
Parts:
- removed D4, D5: XL-1010RGBC-WS2812B, RevK:SMD1010, symbol RevK:WS2812B-1mm
- removed J4: Conn_01x03_Socket, RevK:PinHeader_1x03_P2.54mm, symbol Connector:Conn_01x03_Socket
- removed U8: VEML6040, RevK:VEML6040, symbol RevK:VEML6040
- added C27: 100uF 6.3V, RevK:C_1206, symbol Device:C
- added U2: SCD41, RevK:SCD41, symbol RevK:SCD41
Connections:
- net +3.3V: now also U2.19 (VDDH), U2.7 (VDD)
- net GND: now also C27.1, U2.20 (GND), U2.21 (GND), U2.6 (GND)
- net LED: now also U2.15 (GPIO11); no longer U2.25 (GPIO21)
- net SCL: now also U2.14 (GPIO10), U2.9 (SCL); no longer U2.29 (GPIO34)
- net SDA: now also U2.13 (GPIO9), U2.10 (SDA); no longer U2.30 (GPIO48)
- net VBUS: now also C27.2
- no-connect marks 25 -> 24
Other:
- moved on the sheet: C3, C4, J3, R1, R2
