File: PCB/Env3/EnvMon.kicad_pcb (KiCad board)
At the start: 2 copper layers, 70 x 70 mm, 46 parts, among them J1 LCD, J2 DC, J3 TEMP, J4 LCD, J5 Reset, J6 USB-C-Socket-H, J7 TC2030-USB-NL-DS, U1 ESP32-S3-MINI-1, U2 SCD41, U3 MD8942, U4 MCP9808_MSOP, U5 GZP6816D, U8 VEML6040

Commit message: Tidy up
Routing:
- net GND: track 40.3 -> 49.9 mm
- net LED: track 21.4 -> 20.7 mm

Commit message: render
Routing:
- net GND: track 49.9 -> 55.2 mm
Other:
- board text added: "."
- board text added: "C"

Commit message: tweak
Other:
- board text added: "B"
- board text added: "®"
- board text removed: "AB"
