File: PCB/Env3/EnvMon.kicad_pcb (KiCad board)
At the start: 2 copper layers, 70 x 70 mm, 46 parts, among them J1 LCD, J2 DC, J3 TEMP, J4 LCD, J5 Reset, J6 USB-C-Socket-H, J7 TC2030-USB-NL-DS, U1 ESP32-S3-MINI-1, U2 SCD41, U3 MD8942, U4 MCP9808_MSOP, U5 GZP6816D, U8 VEML6040

Commit message: Library update
Parts:
- J1: footprint RevK:PinSocket_1x08_P2.54mm_Vertical_SMD -> RevK:LCD2
- moved J1 0.10 mm to (73.4, 83.6)

Commit message: As ordered
Parts:
- U4: value MCP9808_MSOP -> TMP1075DSG; footprint Package_SO:MSOP-8_3x3mm_P0.65mm -> Package_SON:WSON-8-1EP_2x2mm_P0.5mm_EP0.9x1.6mm_ThermalVias
- moved C5 11.0 mm to (80.2, 111.2)
- moved C6 6.34 mm to (116.0, 78.2), turned to 0 degrees
- moved U4 1.75 mm to (116.0, 76.5), turned to 180 degrees
- moved U2 0.50 mm to (77.5, 117.0)
- moved J4 0.10 mm to (126.6, 83.4)
Routing:
- net GND: track 55.2 -> 75.1 mm, vias 82 -> 90
- net +3.3V: track 184.0 -> 203.5 mm
- net SDA: track 92.1 -> 95.1 mm
- net SCL: track 102.6 -> 103.5 mm
Other:
- board text added: "TMP1075"
- board text removed: "MCP9808"
- board text removed: "T+H"
