File: PCB/Env3/EnvMon.kicad_sch (KiCad schematic)
At the start: 51 parts, among them J1 LCD, J10 Conn_01x01, J11 Conn_01x01, J12 Conn_01x01, J2 DC, J3 TEMP, J4 LCD, J5 Reset, J6 USB-C-Socket-H, J7 TC2030-USB-NL-DS, J8 T6793, J9 Conn_01x01, U1 ESP32-S3-MINI-1, U2 SCD41, U3 MD8942, U4 MCP9808_MSOP, U5 GZP6816D, U8 VEML6040

Commit message: New board
Parts:
- removed C12: 100nF, RevK:C_0402, symbol Device:C
- removed J10, J11, J12, J9: Conn_01x01, RevK:PinHeader_1x01_P2.54mm_Vertical, symbol Connector_Generic:Conn_01x01
- removed J8: T6793, RevK:PinHeader_1x06_P2.54mm_Vertical, symbol Connector_Generic:Conn_01x06
- added SW1: ~, RevK:Switch-Nav5, symbol RevK:Switch-Nav5
- U2: now fitted; now in the parts list
Connections:
- net GND: now also SW1.5 (COM)
- net LED: now also U1.44 (GPIO46); no longer U1.32 (GPIO36)
- net SCL: now also U1.5 (GPIO1); no longer U1.34 (GPIO38)
- net SDA: now also U1.6 (GPIO2); no longer U1.35 (GPIO39)
- net TEMP: now also U1.31 (GPIO35); no longer U1.16 (GPIO12)
- net N: now reaches U1.33 (GPIO37)
- net N: now also SW1.1 (N)
- net W: now reaches U1.36 (GPIO40)
- net W: now also SW1.3 (W)
- new net E: SW1.4 (E), U1.35 (GPIO39)
- new net P: SW1.2 (PSH), U1.32 (GPIO36)
- new net S: SW1.6 (S), U1.34 (GPIO38)
- now unconnected: U5.2, U5.5, U5.6
- no-connect marks 33 -> 23
Other:
- note removed: "C136710 or C145900 may be good as a button"

Commit message: Library update
Parts:
- J1: footprint RevK:PinSocket_1x08_P2.54mm_Vertical_SMD -> RevK:LCD2
Changed lines of the file:
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@@
 			)
 		)
-		(property "Footprint" "RevK:PinSocket_1x08_P2.54mm_Vertical_SMD"
+		(property "Footprint" "RevK:LCD2"
 			(at 120.65 109.855 0)
 			(effects

Commit message: As ordered
Parts:
- removed U4: MCP9808_MSOP, Package_SO:MSOP-8_3x3mm_P0.65mm, symbol Sensor_Temperature:MCP9808_MSOP
- added U4: TMP1075DSG, Package_SON:WSON-8-1EP_2x2mm_P0.5mm_EP0.9x1.6mm_ThermalVias, symbol Sensor_Temperature:TMP1075DSG
Connections:
- net +3.3V: now also U4.8 (V+)
- net GND: now also U4.4 (GND), U4.5 (A2), U4.6 (A1), U4.7 (A0), U4.9 (EP)
- net SCL: now also U4.2 (SCL)
- net SDA: now also U4.1 (SDA)
Other:
- note added: "I2C addresses (hex) 10 VEML6040 18 MCP9808 78 GZP6816D 62 SCD41 15 T6793 48 TMP1075"
- moved on the sheet: C6, C9, U5
