File: PCB/Env2/EnvMon.kicad_sch (KiCad schematic)
At the start: 51 parts, among them J1 LCD, J10 Conn_01x01, J11 Conn_01x01, J12 Conn_01x01, J2 DC, J3 TEMP, J4 LCD, J5 Reset, J6 USB-C-Socket-H, J7 TC2030-USB-NL-DS, J8 T6793, J9 Conn_01x01, U1 ESP32-S3-MINI-1, U2 SCD41, U3 MD8942, U4 MCP9808_MSOP, U5 GZP6816D, U8 VEML6040

Commit message: STL
Parts:
- U2: now fitted; now in the parts list
Changed lines of the file:
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@@
 		(unit 1)
 		(exclude_from_sim no)
-		(in_bom no)
+		(in_bom yes)
 		(on_board yes)
-		(dnp yes)
+		(dnp no)
 		(fields_autoplaced yes)
 		(property "Reference" "U2"

Commit message: Library update
Parts:
- J1: footprint RevK:PinSocket_1x08_P2.54mm_Vertical_SMD -> RevK:LCD2
Changed lines of the file:
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@@
 			)
 		)
-		(property "Footprint" "RevK:PinSocket_1x08_P2.54mm_Vertical_SMD"
+		(property "Footprint" "RevK:LCD2"
 			(at 120.65 109.855 0)
 			(effects

Commit message: As ordered
Other:
- note removed: "C136710 or C145900 may be good as a button"
Changed lines of the file:
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@@
 		(comment 2 "www.me.uk")
-	)
-	(text "C136710 or C145900 may be good as a button"
-		(exclude_from_sim no)
-		(at 251.46 156.21 0)
-		(effects
-			(font
-				(size 1.27 1.27)
-			)
-		)
 	)
 	(junction

Commit message: Moved to FaikinRemote project
Parts:
- D4: footprint RevK:SMD1010 -> RevK:SMD1010-Side
- U8: footprint RevK:VEML6040 -> RevK:VEML6040-Side
Changed lines of the file:
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@@
 			)
 		)
-		(property "Footprint" "RevK:SMD1010"
+		(property "Footprint" "RevK:SMD1010-Side"
 			(at 162.56 43.815 0)
 			(effects
@@
 			)
 		)
-		(property "Footprint" "RevK:VEML6040"
+		(property "Footprint" "RevK:VEML6040-Side"
 			(at 254 126.365 0)
 			(effects

Commit message: New case work
Parts:
- D4: footprint RevK:SMD1010-Side -> RevK:SMD1010-Side2
- U4: footprint Package_SO:MSOP-8_3x3mm_P0.65mm -> RevK:MSOP-8_3x3mm_P0.65mm-SIde
Changed lines of the file:
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@@
 			)
 		)
-		(property "Footprint" "RevK:SMD1010-Side"
+		(property "Footprint" "RevK:SMD1010-Side2"
 			(at 162.56 43.815 0)
 			(effects
@@
 			)
 		)
-		(property "Footprint" "Package_SO:MSOP-8_3x3mm_P0.65mm"
+		(property "Footprint" "RevK:MSOP-8_3x3mm_P0.65mm-SIde"
 			(at 253.365 109.22 0)
 			(effects
